File: V1/Hardware/PCB/Booklight/Booklight.kicad_sch (KiCad schematic)
At the start: 34 parts, among them J1 Alterative_charging, Q2 8205A, U1 TP4056-42-ESOP8, U3 DW01A, U7 MCP1825S, U8 LM397

Commit message: Swapped comperator
Parts:
- removed U8: LM397, Package_TO_SOT_SMD:SOT-23-5, symbol Comparator:LM397
- added U3: TLV7041DBV, Package_TO_SOT_SMD:SOT-23-5, symbol Comparator:TLV7041DBV
- R3: renamed from R11; value 1k -> 2k
- renumbered C8 to C1, C12 to C2, C13 to C3, C20 to C4, C11 to C5, C17 to C6, C18 to C7, C19 to C8, Q2 to Q1, R16 to R10, R20 to R11, R22 to R12, R21 to R13, R12 to R4, R13 to R5, R14 to R6, R19 to R7, R15 to R8, R17 to R9, U3 to U2, U7 to U4
Connections:
- net 3.3V: now also U3.5 (V+)
- net GND: now also U3.2 (V-)
- net Ref: now also U3.4 (-)
- net at R10.2: now also U3.3 (+)
- net at D3.2 (A), R11.1: now also U3.1
